File: boot_camp_pcb/boot_camp_pcb.kicad_pcb (KiCad board)
At the start: 2 copper layers, 101.6 x 101.6 mm, 32 parts, among them J1 Screw_Terminal_01x02, M2 Fan, Q1 NMOS, SW1 SW_SPST, SW2 SW_Push, SW3 SW_Push, U1 DHT20, U2 LM7805_TO220

Commit message: finish pcb, make demo
Parts:
- added J2: Conn_01x06, Connector_PinHeader_2.54mm:PinHeader_1x06_P2.54mm_Vertical, F.Cu at (84.5, 138.4)
- added R10: 470, Resistor_SMD:R_0805_2012Metric, F.Cu at (89.3, 74.9)
- added R11: 470, Resistor_SMD:R_0805_2012Metric, F.Cu at (110.6, 74.8)
- Q1: value NMOS -> Q_NMOS_GDS
- moved LS1 15.4 mm to (125.0, 118.1)
- moved R5 13.9 mm to (75.9, 128.9), turned to 90 degrees
- moved R4 11.7 mm to (79.4, 128.9), turned to 90 degrees
- moved A1 10.2 mm to (66.7, 122.6)
- moved R7 1.68 mm to (57.8, 45.1), turned to 180 degrees
- moved Q1 0.90 mm to (126.5, 74.7)
- turned R3 to 180 degrees
Connections:
- D2 pad 2: Net-(A1-D8) -> Net-(D2-A)
- D3 pad 2: Net-(A1-D9) -> Net-(D3-A)
- Q1 pad 1: Net-(M2--) -> Net-(A1-D10)
- Q1 pad 2: Net-(A1-D10) -> Net-(M2--)
Routing:
- net +12V: track 0.00 -> 160.9 mm, vias 0 -> 5
- net /TX: track 0.00 -> 133.5 mm, vias 0 -> 2
- net /SDA: track 0.00 -> 132.4 mm, vias 0 -> 2
- net /SCL: track 0.00 -> 125.6 mm, vias 0 -> 2
- net Net-(A1-A0): track 0.00 -> 97.2 mm, vias 0 -> 2
- net Net-(A1-A1): track 0.00 -> 91.7 mm, vias 0 -> 1
- net Net-(A1-D9): track 0.00 -> 67.3 mm, vias 0 -> 2
- net Net-(A1-D10): track 0.00 -> 64.4 mm, vias 0 -> 1
- net Net-(A1-D5): track 0.00 -> 50.3 mm, vias 0 -> 1
- net Net-(A1-D8): track 0.00 -> 49.4 mm, vias 0 -> 1
- net Net-(A1-D7): track 0.00 -> 45.6 mm
- net Net-(A1-D4): track 0.00 -> 37.5 mm
- net /RX: track 0.00 -> 37.2 mm, vias 0 -> 1
- net Net-(A1-D6): track 0.00 -> 35.6 mm
- net Net-(A1-A2): track 0.00 -> 27.9 mm, vias 0 -> 1
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- added copper zone on B.Cu, net +5V
- added copper zone on F.Cu, net GND
Other:
- board text added: "+12"
- board text added: "12V ON"
- board text added: "5V ON"
- board text added: "BU EPIC"
- board text added: "Boot Camp Board - V1.0 E. Hazen - 11/2023"
- board text added: "GND"
- board text added: "POWER"
- board text added: "Pro Micro 5V"
- board text added: "UART"
