File: boot_camp_pcb/boot_camp_pcb.kicad_sch (KiCad schematic)
At the start: 33 parts, among them J1 Screw_Terminal_01x02, M2 Fan, Q1 NMOS, SW1 SW_SPST, SW2 SW_Push, SW3 SW_Push, U1 DHT20, U2 LM7805_TO220, U3 Arduino pro micro

Commit message: finish pcb, make demo
Parts:
- removed Q1: NMOS, Package_TO_SOT_THT:TO-220-3_Vertical, symbol Simulation_SPICE:NMOS
- added J2: Conn_01x06, Connector_PinHeader_2.54mm:PinHeader_1x06_P2.54mm_Vertical, symbol Connector_Generic:Conn_01x06
- added Q1: Q_NMOS_GDS, Package_TO_SOT_THT:TO-220-3_Vertical, symbol Device:Q_NMOS_GDS
- added R10, R11: 470, Resistor_SMD:R_0805_2012Metric, symbol Device:R_US
Connections:
- net GND: now also J2.1 (Pin_1), Q1.3 (S)
- net RX: now also J2.4 (Pin_4)
- net TX: now also J2.5 (Pin_5)
- net at D3.2 (A): now also R11.1; no longer A1.12 (D9)
- net at M2.2 (-): now also Q1.2 (D)
- net at D2.2 (A): now also R10.1; no longer A1.11 (D8)
- net at A1.13 (D10): now also Q1.1 (G)
- new net: A1.11 (D8), R10.2
- new net: A1.12 (D9), R11.2
Other:
- note added: "FTDI serial"
Changed lines of the file:
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@@
+    (stroke (width 0) (type default))
+  )
+  (wire (pts (xy 102.87 97.79) (xy 102.87 116.84))
     (stroke (width 0) (type default))
   )
@@
     (stroke (width 0) (type default))
   )
+  (wire (pts (xy 105.41 129.54) (xy 105.41 137.16))
+    (stroke (width 0) (type default))
+  )
   (wire (pts (xy 93.98 43.18) (xy 93.98 45.72))
     (stroke (width 0) (type default))
@@
     (stroke (width 0) (type default))
   )
+  (wire (pts (xy 105.41 100.33) (xy 105.41 121.92))
+    (stroke (width 0) (type default))
+  )
   (wire (pts (xy 106.68 82.55) (xy 118.11 82.55))
     (stroke (width 0) (type default))
@@
     (stroke (width 0) (type default))
   )
+  (wire (pts (xy 223.52 156.21) (xy 229.87 156.21))
+    (stroke (width 0) (type default))
+  )
   (wire (pts (xy 157.48 105.41) (xy 157.48 97.79))
     (stroke (width 0) (type default))
   )
+  (wire (pts (xy 223.52 153.67) (xy 229.87 153.67))
+    (stroke (width 0) (type default))
+  )
   (wire (pts (xy 203.2 33.02) (xy 203.2 30.48))
     (stroke (width 0) (type default))
@@
     (stroke (width 0) (type default))
   )
+  (wire (pts (xy 229.87 146.05) (xy 223.52 146.05))
+    (stroke (width 0) (type default))
+  )
   (wire (pts (xy 93.98 46.99) (xy 109.22 46.99))
     (stroke (width 0) (type default))
@@
     (stroke (width 0) (type default))
   )
+  (wire (pts (xy 223.52 146.05) (xy 223.52 147.32))
+    (stroke (width 0) (type default))
+  )
   (wire (pts (xy 73.66 35.56) (xy 78.74 35.56))
     (stroke (width 0) (type default))
   )
-  (wire (pts (xy 105.41 137.16) (xy 105.41 100.33))
+  (wire (pts (xy 102.87 124.46) (xy 102.87 130.81))
     (stroke (width 0) (type default))
   )
@@
   )
   (wire (pts (xy 160.02 71.12) (xy 160.02 73.66))
-    (stroke (width 0) (type default))
-  )
-  (wire (pts (xy 102.87 130.81) (xy 102.87 97.79))
     (stroke (width 0) (type default))
   )
@@
     (effects (font (size 1.27 1.27)) (justify left bottom))
   )
+  (text "FTDI serial" (at 240.03 147.32 0)
+    (effects (font (size 1.27 1.27)) (justify left bottom))
+  )
   (text "Boston University EPIC" (at 160.02 177.8 0)
     (effects (font (size 3.175 3.175)) (justify left bottom))
@@
     (effects (font (size 1.27 1.27)) (justify left bottom))
   )
+  (label "RX" (at 223.52 153.67 0) (fields_autoplaced)
+    (effects (font (size 1.27 1.27)) (justify left bottom))
+  )
   (label "TX" (at 106.68 80.01 0) (fields_autoplaced)
     (effects (font (size 1.27 1.27)) (justify left bottom))
@@
     (effects (font (size 1.27 1.27)) (justify left bottom))
   )
+  (label "TX" (at 223.52 156.21 0) (fields_autoplaced)
+    (effects (font (size 1.27 1.27)) (justify left bottom))
+  )
   (label "RX" (at 106.68 77.47 0) (fields_autoplaced)
     (effects (font (size 1.27 1.27)) (justify left bottom))
@@
         (path "/af1c231b-dc74-4380-b8ae-be71463061e8"
           (reference "R1") (unit 1)
+        )
+      )
+    )
+  )
+  (symbol (lib_id "Device:R_US") (at 102.87 120.65 180) (unit 1)
+    (in_bom yes) (on_board yes) (dnp no)
+    (property "Reference" "R10" (at 96.52 119.38 0)
+      (effects (font (size 1.27 1.27)) (justify right))
+    )
+    (property "Value" "470" (at 96.52 121.92 0)
+      (effects (font (size 1.27 1.27)) (justify right))
+    )
+    (property "Footprint" "Resistor_SMD:R_0805_2012Metric" (at 101.854 120.396 90)
+      (effects (font (size 1.27 1.27)) hide)
+    )
+    (property "Datasheet" "~" (at 102.87 120.65 0)
+      (effects (font (size 1.27 1.27)) hide)
+    )
+    (pin "1")
+    (pin "2")
+    (instances
+      (project "boot_camp_pcb"
+        (path "/af1c231b-dc74-4380-b8ae-be71463061e8"
+          (reference "R10") (unit 1)
+        )
+      )
+    )
+  )
+  (symbol (lib_id "Connector_Generic:Conn_01x06") (at 234.95 151.13 0) (unit 1)
+    (in_bom yes) (on_board yes) (dnp no) (fields_autoplaced)
+    (property "Reference" "J2" (at 237.49 151.13 0)
+      (effects (font (size 1.27 1.27)) (justify left))
+    )
+    (property "Value" "Conn_01x06" (at 237.49 153.67 0)
+      (effects (font (size 1.27 1.27)) (justify left))
+    )
+    (property "Footprint" "Connector_PinHeader_2.54mm:PinHeader_1x06_P2.54mm_Vertical" (at 234.95 151.13 0)
+      (effects (font (size 1.27 1.27)) hide)
+    )
+    (property "Datasheet" "~" (at 234.95 151.13 0)
+      (effects (font (size 1.27 1.27)) hide)
+    )
+    (property "MfgNo" "68001-106HLF" (at 234.95 151.13 0)
+      (effects (font (size 1.27 1.27)) hide)
+    )
+    (property "CatNo" "609-3272-ND" (at 234.95 151.13 0)
+      (effects (font (size 1.27 1.27)) hide)
+    )
+    (property "Type" "TH" (at 234.95 151.13 0)
+      (effects (font (size 1.27 1.27)) hide)
+    )
+    (pin "1")
+    (pin "2")
+    (pin "3")
+    (pin "4")
+    (pin "5")
+    (pin "6")
+    (instances
+      (project "boot_camp_pcb"
+        (path "/af1c231b-dc74-4380-b8ae-be71463061e8"
+          (reference "J2") (unit 1)
+        )
+      )
+      (project "iso-master-fmc"
+        (path "/c16c7191-fd02-4980-bf49-c35772663650"
+          (reference "J4") (unit 1)
+        )
+      )
+    )
+  )
+  (symbol (lib_id "Device:R_US") (at 105.41 125.73 0) (mirror x) (unit 1)
+    (in_bom yes) (on_board yes) (dnp no)
+    (property "Reference" "R11" (at 111.76 124.46 0)
+      (effects (font (size 1.27 1.27)) (justify right))
+    )
+    (property "Value" "470" (at 111.76 127 0)
+      (effects (font (size 1.27 1.27)) (justify right))
+    )
+    (property "Footprint" "Resistor_SMD:R_0805_2012Metric" (at 106.426 125.476 90)
+      (effects (font (size 1.27 1.27)) hide)
+    )
+    (property "Datasheet" "~" (at 105.41 125.73 0)
+      (effects (font (size 1.27 1.27)) hide)
+    )
+    (pin "1")
+    (pin "2")
+    (instances
+      (project "boot_camp_pcb"
+        (path "/af1c231b-dc74-4380-b8ae-be71463061e8"
+          (reference "R11") (unit 1)
         )
       )
@@
     )
   )
+  (symbol (lib_id "Device:Q_NMOS_GDS") (at 157.48 154.94 0) (unit 1)
+    (in_bom yes) (on_board yes) (dnp no) (fields_autoplaced)
+    (property "Reference" "Q1" (at 163.83 153.67 0)
+      (effects (font (size 1.27 1.27)) (justify left))
+    )
+    (property "Value" "Q_NMOS_GDS" (at 163.83 156.21 0)
+      (effects (font (size 1.27 1.27)) (justify left))
+    )
+    (property "Footprint" "Package_TO_SOT_THT:TO-220-3_Vertical" (at 162.56 152.4 0)
+      (effects (font (size 1.27 1.27)) hide)
+    )
+    (property "Datasheet" "~" (at 157.48 154.94 0)
+      (effects (font (size 1.27 1.27)) hide)
+    )
+    (pin "1")
+    (pin "2")
+    (pin "3")
+    (instances
+      (project "boot_camp_pcb"
+        (path "/af1c231b-dc74-4380-b8ae-be71463061e8"
+          (reference "Q1") (unit 1)
+        )
+      )
+    )
+  )
   (symbol (lib_id "Mechanical:MountingHole") (at 19.05 151.13 0) (unit 1)
     (in_bom yes) (on_board yes) (dnp no) (fields_autoplaced)
@@
         (path "/af1c231b-dc74-4380-b8ae-be71463061e8"
           (reference "H4") (unit 1)
+        )
+      )
+    )
+  )
+  (symbol (lib_id "power:GND") (at 223.52 147.32 0) (unit 1)
+    (in_bom yes) (on_board yes) (dnp no)
+    (property "Reference" "#PWR024" (at 223.52 153.67 0)
+      (effects (font (size 1.27 1.27)) hide)
+    )
+    (property "Value" "GND" (at 226.06 147.32 0)
+      (effects (font (size 1.27 1.27)))
+    )
+    (property "Footprint" "" (at 223.52 147.32 0)
+      (effects (font (size 1.27 1.27)) hide)
+    )
+    (property "Datasheet" "" (at 223.52 147.32 0)
+      (effects (font (size 1.27 1.27)) hide)
+    )
+    (pin "1")
+    (instances
+      (project "boot_camp_pcb"
+        (path "/af1c231b-dc74-4380-b8ae-be71463061e8"
+          (reference "#PWR024") (unit 1)
+        )
+      )
+      (project "iso-master-fmc"
+        (path "/c16c7191-fd02-4980-bf49-c35772663650"
+          (reference "#PWR058") (unit 1)
         )
       )
@@
         )
       )
-    )
-  )
-  (symbol (lib_id "Simulation_SPICE:NMOS") (at 157.48 154.94 0) (unit 1)
-    (in_bom yes) (on_board yes) (dnp no)
-    (property "Reference" "Q1" (at 163.83 153.67 0)
-      (effects (font (size 1.27 1.27)) (justify left))
-    )
-    (property "Value" "NMOS" (at 163.83 156.21 0)
-      (effects (font (size 1.27 1.27)) (justify left))
-    )
-    (property "Footprint" "Package_TO_SOT_THT:TO-220-3_Vertical" (at 162.56 152.4 0)
-      (effects (font (size 1.27 1.27)) hide)
-    )
-    (property "Datasheet" "https://ngspice.sourceforge.io/docs/ngspice-manual.pdf" (at 157.48 167.64 0)
-      (effects (font (size 1.27 1.27)) hide)
-    )
-    (property "Sim.Device" "NMOS" (at 157.48 172.085 0)
-      (effects (font (size 1.27 1.27)) hide)
-    )
-    (property "Sim.Type" "VDMOS" (at 157.48 173.99 0)
-      (effects (font (size 1.27 1.27)) hide)
-    )
-    (property "Sim.Pins" "1=D 2=G 3=S" (at 157.48 170.18 0)
-      (effects (font (size 1.27 1.27)) hide)
-    )
-    (property "CatNo" "497-2757-5-ND" (at 171.45 160.02 0)
-      (effects (font (size 1.27 1.27)))
-    )
-    (pin "1")
-    (pin "2")
-    (pin "3")
-    (instances
-      (project "boot_camp_pcb"
-        (path "/af1c231b-dc74-4380-b8ae-be71463061e8"
-          (reference "Q1") (unit 1)
-        )
-      )
