File: tiny-avr/tiny-avr.kicad_pcb (KiCad board)
At the start: 2 copper layers, 19 x 31.8 mm, 21 parts, among them J1 Conn_01x12, J2 Conn_01x12, J3 USB_B_Micro, U1 ATtiny1606-M, U2 FT232RL

Commit message: working on tiny
Parts:
- removed U1: ATtiny1606-M, Package_DFN_QFN:VQFN-20-1EP_3x3mm_P0.4mm_EP1.7x1.7mm
- added U3: ATtiny1606-S, Package_SO:SOIC-20W_7.5x12.8mm_P1.27mm, F.Cu at (78.5, 42.1)
- moved D1 19.7 mm to (56.1, 48.1)
- moved D2 19.7 mm to (56.1, 46.2)
- moved D3 19.7 mm to (62.0, 48.1)
- moved R2 19.7 mm to (62.0, 45.6)
- moved R3 19.7 mm to (56.1, 47.6)
- moved R4 19.7 mm to (56.1, 45.6)
- moved R5 19.7 mm to (62.0, 47.5)
- moved C1 18.4 mm to (60.6, 37.6)
Routing:
- net /PB3: track 7.31 -> 0.00 mm
