File: tiny-avr/tiny-avr.kicad_sch (KiCad schematic)
At the start: 21 parts, among them J1 Conn_01x12, J2 Conn_01x12, J3 USB_B_Micro, U1 ATtiny1606-M, U2 FT232RL

Commit message: working on tiny
Parts:
- removed U1: ATtiny1606-M, Package_DFN_QFN:VQFN-20-1EP_3x3mm_P0.4mm_EP1.7x1.7mm, symbol MCU_Microchip_ATtiny:ATtiny1606-M
- added U3: ATtiny1606-S, Package_SO:SOIC-20W_7.5x12.8mm_P1.27mm, symbol MCU_Microchip_ATtiny:ATtiny1606-S
Connections:
- net GND: now also U3.20 (GND)
- net PB2: now also U3.16 (~{RESET}/PA0)
- net PB3: now also U3.8 (PB3)
- net PB4: now also U3.7 (PB4)
- net PB5: now also U3.6 (PB5)
- net VCC: now also U3.1 (VCC)
- net at J2.10 (Pin_10): now also U3.14 (PC2)
- net at J2.11 (Pin_11): now also U3.15 (PC3)
- net at J2.8 (Pin_8), R5.1: now also U3.12 (PC0)
- net at J2.9 (Pin_9): now also U3.13 (PC1)
- net at J1.10 (Pin_10): now also U3.11 (PB0)
- net at J1.11 (Pin_11): now also U3.10 (PB1)
- net at J1.12 (Pin_12): now also U3.9 (PB2)
- net at J1.3 (Pin_3): now also U3.17 (PA1)
- net at J1.4 (Pin_4): now also U3.18 (PA2)
- net at J1.5 (Pin_5): now also U3.19 (PA3)
- net at J1.6 (Pin_6): now also U3.2 (PA4)
- net at J1.7 (Pin_7): now also U3.3 (PA5)
- net at J1.8 (Pin_8): now also U3.4 (PA6)
- net at J1.9 (Pin_9): now also U3.5 (PA7)
Changed lines of the file:
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@@
+	)
+	(symbol
+		(lib_id "MCU_Microchip_ATtiny:ATtiny1606-S")
+		(at 204.47 83.82 0)
+		(unit 1)
+		(exclude_from_sim no)
+		(in_bom yes)
+		(on_board yes)
+		(dnp no)
+		(fields_autoplaced yes)
+		(property "Reference" "U3"
+			(at 206.6133 58.42 0)
+			(effects
+				(font
+					(size 1.27 1.27)
+				)
+				(justify left)
+			)
+		)
+		(property "Value" "ATtiny1606-S"
+			(at 206.6133 60.96 0)
+			(effects
+				(font
+					(size 1.27 1.27)
+				)
+				(justify left)
+			)
+		)
+		(property "Footprint" "Package_SO:SOIC-20W_7.5x12.8mm_P1.27mm"
+			(at 204.47 83.82 0)
+			(effects
+				(font
+					(size 1.27 1.27)
+					(italic yes)
+				)
+				(hide yes)
+			)
+		)
+		(property "Datasheet" "http://ww1.microchip.com/downloads/en/DeviceDoc/ATtiny806_1606_Data_Sheet_40002029A.pdf"
+			(at 204.47 83.82 0)
+			(effects
+				(font
+					(size 1.27 1.27)
+				)
+				(hide yes)
+			)
+		)
+		(property "Description" "20MHz, 16kB Flash, 1kB SRAM, 256B EEPROM, SOIC-20"
+			(at 204.47 83.82 0)
+			(effects
+				(font
+					(size 1.27 1.27)
+				)
+				(hide yes)
+			)
+		)
+		(pin "17"
+		)
+		(pin "16"
+		)
+		(pin "10"
+		)
+		(pin "1"
+		)
+		(pin "13"
+		)
+		(pin "15"
+		)
+		(pin "14"
+		)
+		(pin "12"
+		)
+		(pin "6"
+		)
+		(pin "19"
+		)
+		(pin "4"
+		)
+		(pin "3"
+		)
+		(pin "5"
+		)
+		(pin "9"
+		)
+		(pin "8"
+		)
+		(pin "7"
+		)
+		(pin "11"
+		)
+		(pin "18"
+		)
+		(pin "20"
+		)
+		(pin "2"
+		)
+		(instances
+			(project ""
+				(path "/345db647-d2f4-43e4-9b06-9f1535b9a87c"
+					(reference "U3")
+					(unit 1)
+				)
+			)
+		)
 	)
 	(symbol
@@
 					(unit 1)
 				)
-			)
-		)
-	)
-	(symbol
-		(lib_id "MCU_Microchip_ATtiny:ATtiny1606-M")
-		(at 204.47 83.82 0)
-		(unit 1)
-		(exclude_from_sim no)
-		(in_bom yes)
-		(on_board yes)
-		(dnp no)
-		(property "Reference" "U1"
-			(at 206.6133 58.42 0)
-			(effects
-				(font
-					(size 1.27 1.27)
-				)
-				(justify left)
-			)
-		)
-		(property "Value" "ATtiny1606-M"
-			(at 206.6133 60.96 0)
-			(effects
-				(font
-					(size 1.27 1.27)
-				)
-				(justify left)
-			)
-		)
-		(property "Footprint" "Package_DFN_QFN:VQFN-20-1EP_3x3mm_P0.4mm_EP1.7x1.7mm"
-			(at 204.47 83.82 0)
-			(effects
-				(font
-					(size 1.27 1.27)
-					(italic yes)
-				)
-				(hide yes)
-			)
-		)
-		(property "Datasheet" "http://ww1.microchip.com/downloads/en/DeviceDoc/ATtiny806_1606_Data_Sheet_40002029A.pdf"
-			(at 204.47 83.82 0)
-			(effects
-				(font
-					(size 1.27 1.27)
-				)
-				(hide yes)
-			)
-		)
-		(property "Description" "20MHz, 16kB Flash, 1kB SRAM, 256B EEPROM, VQFN-20"
-			(at 204.47 83.82 0)
-			(effects
-				(font
-					(size 1.27 1.27)
-				)
-				(hide yes)
-			)
-		)
-		(property "CatNo" "150-ATTINY1606-MNRCT-ND"
-			(at 221.996 105.664 0)
-			(effects
-				(font
-					(size 1.27 1.27)
-				)
-			)
-		)
-		(property "MfgNo" "ATTINY1606-MNR"
-			(at 204.47 83.82 0)
-			(effects
-				(font
-					(size 1.27 1.27)
-				)
-				(hide yes)
-			)
-		)
-		(pin "8"
-		)
-		(pin "5"
-		)
-		(pin "2"
-		)
-		(pin "6"
-		)
-		(pin "13"
-		)
-		(pin "12"
-		)
-		(pin "9"
-		)
-		(pin "11"
-		)
-		(pin "7"
-		)
-		(pin "10"
-		)
-		(pin "4"
-		)
-		(pin "3"
-		)
-		(pin "1"
-		)
-		(pin "14"
-		)
-		(pin "18"
-		)
-		(pin "21"
-		)
-		(pin "17"
-		)
-		(pin "16"
-		)
-		(pin "15"
-		)
-		(pin "19"
-		)
-		(pin "20"
-		)
-		(instances
-			(project ""
-				(path "/345db647-d2f4-43e4-9b06-9f1535b9a87c"
-					(reference "U1")
-					(unit 1)
-				)
